File: hw/mini-macro-keyboard-eco/mini-macro-keyboard-eco.sch (KiCad schematic (older format))
At the start: 39 parts, among them J0 USB_B_Micro, J1 SWD, SW0 SW_SPDT, SW1 SW_1, SW2 SW_2, SW3 SW_3, SW4 RESET, SW5 SW_SPDT, SW6 SW_SPDT, U1 USBLC6-2SC6, U2 XC6206P322MR, U3 STM32F070F6Px, Y1 16 MHz

Commit message: chore(hw): rescue eco schematic
New version of the kicad is used

Signed-off-by: Ivan Kovalenko <s1ckretbox@gmail.com>
Parts:
- C0, C1, C10, C11, C2, C3, C4, C5, C6, C7, C8, C9: symbol Device:C_Small -> mini-macro-keyboard-eco-rescue:C_Small-Device
- D1, D2, D3: symbol Device:LED_Small -> mini-macro-keyboard-eco-rescue:LED_Small-Device
- J0: symbol Connector:USB_B_Micro -> mini-macro-keyboard-eco-rescue:USB_B_Micro-Connector
- J1: symbol Connector:Conn_01x04_Male -> mini-macro-keyboard-eco-rescue:Conn_01x04_Male-Connector
- R0, R1, R11, R12, R13, R2, R3, R4, R5, R6, R7: symbol Device:R_Small -> mini-macro-keyboard-eco-rescue:R_Small-Device
- SW0, SW5, SW6: symbol Switch:SW_SPDT -> mini-macro-keyboard-eco-rescue:SW_SPDT-Switch
- SW1, SW2, SW3, SW4: symbol Switch:SW_Push -> mini-macro-keyboard-eco-rescue:SW_Push-Switch
- U1: symbol Power_Protection:USBLC6-2SC6 -> mini-macro-keyboard-eco-rescue:USBLC6-2SC6-Power_Protection
- U2: symbol Regulator_Linear:XC6206PxxxMR -> mini-macro-keyboard-eco-rescue:XC6206PxxxMR-Regulator_Linear
- U3: symbol MCU_ST_STM32F0:STM32F070F6Px -> mini-macro-keyboard-eco-rescue:STM32F070F6Px-MCU_ST_STM32F0
- Y1: symbol Device:Crystal_GND24_Small -> mini-macro-keyboard-eco-rescue:Crystal_GND24_Small-Device

Commit message: feat(hw): assign footprints
Signed-off-by: Ivan Kovalenko <s1ckretbox@gmail.com>
Parts:
- C0, C1, C10, C11, C2, C3, C4, C5, C6, C7, C8, C9: footprint (none) -> Capacitor_SMD:C_0402_1005Metric
- D1, D2, D3: footprint (none) -> LED_SMD:LED_0603_1608Metric
- J0: footprint (none) -> Connector_USB:USB_Micro-B_Molex-105017-0001
- J1: footprint (none) -> Connector_PinHeader_2.54mm:PinHeader_1x04_P2.54mm_Horizontal
- R0, R1, R2, R3, R4, R5, R6, R7: footprint (none) -> Resistor_SMD:R_0402_1005Metric
- R11, R12, R13: footprint (none) -> Resistor_SMD:R_0603_1608Metric
- SW0, SW5, SW6: footprint (none) -> Button_Switch_SMD:SW_SPDT_PCM12
- SW1, SW2, SW3: footprint (none) -> Button_Switch_Keyboard:SW_Cherry_MX_1.00u_PCB
- SW4: footprint (none) -> Button_Switch_THT:SW_PUSH_6mm
- Y1: footprint (none) -> Crystal:Crystal_SMD_3225-4Pin_3.2x2.5mm
Changed lines of the file:
@@
 F 0 "C5" H 3400 1250 50  0000 L CNN
 F 1 "100n" H 3350 1150 50  0000 L CNN
-F 2 "" H 3300 1200 50  0001 C CNN
+F 2 "Capacitor_SMD:C_0402_1005Metric" H 3300 1200 50  0001 C CNN
 F 3 "~" H 3300 1200 50  0001 C CNN
 	1    3300 1200
@@
 F 0 "C6" H 3700 1250 50  0000 L CNN
 F 1 "100n" H 3650 1150 50  0000 L CNN
-F 2 "" H 3600 1200 50  0001 C CNN
+F 2 "Capacitor_SMD:C_0402_1005Metric" H 3600 1200 50  0001 C CNN
 F 3 "~" H 3600 1200 50  0001 C CNN
 	1    3600 1200
@@
 F 0 "C4" H 1600 1550 50  0000 L CNN
 F 1 "100n" H 1550 1450 50  0000 L CNN
-F 2 "" H 1500 1500 50  0001 C CNN
+F 2 "Capacitor_SMD:C_0402_1005Metric" H 1500 1500 50  0001 C CNN
 F 3 "~" H 1500 1500 50  0001 C CNN
 	1    1500 1500
@@
 F 0 "C7" H 4050 1250 50  0000 L CNN
 F 1 "4.7u" H 4000 1150 50  0000 L CNN
-F 2 "" H 3950 1200 50  0001 C CNN
+F 2 "Capacitor_SMD:C_0402_1005Metric" H 3950 1200 50  0001 C CNN
 F 3 "~" H 3950 1200 50  0001 C CNN
 	1    3950 1200
@@
 F 0 "C9" H 950 4700 50  0000 L CNN
 F 1 "12p" H 950 4800 50  0000 L CNN
-F 2 "" H 1200 4750 50  0001 C CNN
+F 2 "Capacitor_SMD:C_0402_1005Metric" H 1200 4750 50  0001 C CNN
 F 3 "~" H 1200 4750 50  0001 C CNN
 	1    1200 4750
@@
 F 0 "R4" V 1600 1100 50  0000 C CNN
 F 1 "10k" V 1400 1100 50  0000 C CNN
-F 2 "" H 1500 1100 50  0001 C CNN
+F 2 "Resistor_SMD:R_0402_1005Metric" H 1500 1100 50  0001 C CNN
 F 3 "~" H 1500 1100 50  0001 C CNN
 	1    1500 1100
@@
 F 0 "R7" H 1900 4200 50  0000 C CNN
 F 1 "47" H 1900 4100 50  0000 C CNN
-F 2 "" H 1750 4150 50  0001 C CNN
+F 2 "Resistor_SMD:R_0402_1005Metric" H 1750 4150 50  0001 C CNN
 F 3 "~" H 1750 4150 50  0001 C CNN
 	1    1750 4150
@@
 F 0 "J0" H 1057 7067 50  0000 C CNN
 F 1 "USB_B_Micro" H 1057 6976 50  0000 C CNN
-F 2 "" H 1150 6550 50  0001 C CNN
+F 2 "Connector_USB:USB_Micro-B_Molex-105017-0001" H 1150 6550 50  0001 C CNN
 F 3 "~" H 1150 6550 50  0001 C CNN
 	1    1000 6600
@@
 F 0 "D1" H 7900 800 50  0000 C CNN
 F 1 "BLUE" H 7900 1050 50  0000 C CNN
-F 2 "" V 7900 900 50  0001 C CNN
+F 2 "LED_SMD:LED_0603_1608Metric" V 7900 900 50  0001 C CNN
 F 3 "~" V 7900 900 50  0001 C CNN
 	1    7900 900
@@
 F 0 "R11" V 8350 900 50  0000 C CNN
 F 1 "330" V 8150 900 50  0000 C CNN
-F 2 "" H 8250 900 50  0001 C CNN
+F 2 "Resistor_SMD:R_0603_1608Metric" H 8250 900 50  0001 C CNN
 F 3 "~" H 8250 900 50  0001 C CNN
 	1    8250 900
@@
 F 0 "D2" H 7900 1150 50  0000 C CNN
 F 1 "BLUE" H 7900 1400 50  0000 C CNN
-F 2 "" V 7900 1250 50  0001 C CNN
+F 2 "LED_SMD:LED_0603_1608Metric" V 7900 1250 50  0001 C CNN
 F 3 "~" V 7900 1250 50  0001 C CNN
 	1    7900 1250
@@
 F 0 "R12" V 8350 1250 50  0000 C CNN
 F 1 "330" V 8150 1250 50  0000 C CNN
-F 2 "" H 8250 1250 50  0001 C CNN
+F 2 "Resistor_SMD:R_0603_1608Metric" H 8250 1250 50  0001 C CNN
 F 3 "~" H 8250 1250 50  0001 C CNN
 	1    8250 1250
@@
 F 0 "D3" H 7900 1500 50  0000 C CNN
 F 1 "BLUE" H 7900 1750 50  0000 C CNN
-F 2 "" V 7900 1600 50  0001 C CNN
+F 2 "LED_SMD:LED_0603_1608Metric" V 7900 1600 50  0001 C CNN
 F 3 "~" V 7900 1600 50  0001 C CNN
 	1    7900 1600
@@
 F 0 "R13" V 8350 1600 50  0000 C CNN
 F 1 "330" V 8150 1600 50  0000 C CNN
-F 2 "" H 8250 1600 50  0001 C CNN
+F 2 "Resistor_SMD:R_0603_1608Metric" H 8250 1600 50  0001 C CNN
 F 3 "~" H 8250 1600 50  0001 C CNN
 	1    8250 1600
@@
 F 0 "C0" H 9800 1250 50  0000 L CNN
 F 1 "100n" H 9750 1150 50  0000 L CNN
-F 2 "" H 9700 1200 50  0001 C CNN
+F 2 "Capacitor_SMD:C_0402_1005Metric" H 9700 1200 50  0001 C CNN
 F 3 "~" H 9700 1200 50  0001 C CNN
 	1    9700 1200
@@
 F 0 "SW4" V 1400 1700 50  0000 R CNN
 F 1 "RESET" V 1100 1850 50  0000 R CNN
-F 2 "" H 1250 1700 50  0001 C CNN
+F 2 "Button_Switch_THT:SW_PUSH_6mm" H 1250 1700 50  0001 C CNN
 F 3 "~" H 1250 1700 50  0001 C CNN
 	1    1250 1500
@@
 F 0 "SW1" V 5700 3300 50  0000 R CNN
 F 1 "SW_1" V 5400 3450 50  0000 R CNN
-F 2 "" H 5550 3300 50  0001 C CNN
+F 2 "Button_Switch_Keyboard:SW_Cherry_MX_1.00u_PCB" H 5550 3300 50  0001 C CNN
 F 3 "~" H 5550 3300 50  0001 C CNN
 	1    5550 3100
@@
 F 0 "R1" V 5900 2700 50  0000 C CNN
 F 1 "10k" V 5700 2700 50  0000 C CNN
-F 2 "" H 5800 2700 50  0001 C CNN
+F 2 "Resistor_SMD:R_0402_1005Metric" H 5800 2700 50  0001 C CNN
 F 3 "~" H 5800 2700 50  0001 C CNN
 	1    5800 2700
@@
 F 0 "C1" H 5900 3150 50  0000 L CNN
 F 1 "100n" H 5850 3050 50  0000 L CNN
-F 2 "" H 5800 3100 50  0001 C CNN
+F 2 "Capacitor_SMD:C_0402_1005Metric" H 5800 3100 50  0001 C CNN
 F 3 "~" H 5800 3100 50  0001 C CNN
 	1    5800 3100
@@
 F 0 "SW3" V 8100 3300 50  0000 R CNN
 F 1 "SW_3" V 7800 3450 50  0000 R CNN
-F 2 "" H 7950 3300 50  0001 C CNN
+F 2 "Button_Switch_Keyboard:SW_Cherry_MX_1.00u_PCB" H 7950 3300 50  0001 C CNN
 F 3 "~" H 7950 3300 50  0001 C CNN
 	1    7950 3100
@@
 F 0 "R3" V 8300 2700 50  0000 C CNN
 F 1 "10k" V 8100 2700 50  0000 C CNN
-F 2 "" H 8200 2700 50  0001 C CNN
+F 2 "Resistor_SMD:R_0402_1005Metric" H 8200 2700 50  0001 C CNN
 F 3 "~" H 8200 2700 50  0001 C CNN
 	1    8200 2700
@@
 F 0 "C3" H 8300 3150 50  0000 L CNN
 F 1 "100n" H 8250 3050 50  0000 L CNN
-F 2 "" H 8200 3100 50  0001 C CNN
+F 2 "Capacitor_SMD:C_0402_1005Metric" H 8200 3100 50  0001 C CNN
 F 3 "~" H 8200 3100 50  0001 C CNN
 	1    8200 3100
@@
 F 0 "SW2" V 6900 3300 50  0000 R CNN
 F 1 "SW_2" V 6600 3450 50  0000 R CNN
-F 2 "" H 6750 3300 50  0001 C CNN
+F 2 "Button_Switch_Keyboard:SW_Cherry_MX_1.00u_PCB" H 6750 3300 50  0001 C CNN
 F 3 "~" H 6750 3300 50  0001 C CNN
 	1    6750 3100
@@
 F 0 "R2" V 7100 2700 50  0000 C CNN
 F 1 "10k" V 6900 2700 50  0000 C CNN
-F 2 "" H 7000 2700 50  0001 C CNN
+F 2 "Resistor_SMD:R_0402_1005Metric" H 7000 2700 50  0001 C CNN
 F 3 "~" H 7000 2700 50  0001 C CNN
 	1    7000 2700
@@
 F 0 "C2" H 7100 3150 50  0000 L CNN
 F 1 "100n" H 7050 3050 50  0000 L CNN
-F 2 "" H 7000 3100 50  0001 C CNN
+F 2 "Capacitor_SMD:C_0402_1005Metric" H 7000 3100 50  0001 C CNN
 F 3 "~" H 7000 3100 50  0001 C CNN
 	1    7000 3100
@@
 F 0 "C10" H 5450 1500 50  0000 L CNN
 F 1 "1u" H 5500 1300 50  0000 L CNN
-F 2 "" H 5400 1400 50  0001 C CNN
+F 2 "Capacitor_SMD:C_0402_1005Metric" H 5400 1400 50  0001 C CNN
 F 3 "~" H 5400 1400 50  0001 C CNN
 	1    5400 1400
@@
 F 0 "C11" H 6350 1500 50  0000 L CNN
 F 1 "1u" H 6400 1300 50  0000 L CNN
-F 2 "" H 6300 1400 50  0001 C CNN
+F 2 "Capacitor_SMD:C_0402_1005Metric" H 6300 1400 50  0001 C CNN
 F 3 "~" H 6300 1400 50  0001 C CNN
 	1    6300 1400
@@
 F 0 "J1" H 10472 1124 50  0000 R CNN
 F 1 "SWD" H 10472 1033 50  0000 R CNN
-F 2 "" H 10500 1150 50  0001 C CNN
+F 2 "Connector_PinHeader_2.54mm:PinHeader_1x04_P2.54mm_Horizontal" H 10500 1150 50  0001 C CNN
 F 3 "~" H 10500 1150 50  0001 C CNN
 	1    10500 1150
@@
 F 0 "Y1" H 1450 4850 50  0000 L CNN
 F 1 "16 MHz" H 1350 4750 50  0000 L CNN
-F 2 "" H 1500 4500 50  0001 C CNN
+F 2 "Crystal:Crystal_SMD_3225-4Pin_3.2x2.5mm" H 1500 4500 50  0001 C CNN
 F 3 "~" H 1500 4500 50  0001 C CNN
 	1    1500 4500
@@
 F 0 "C8" H 1550 4700 50  0000 L CNN
 F 1 "12p" H 1500 4800 50  0000 L CNN
-F 2 "" H 1750 4750 50  0001 C CNN
+F 2 "Capacitor_SMD:C_0402_1005Metric" H 1750 4750 50  0001 C CNN
 F 3 "~" H 1750 4750 50  0001 C CNN
 	1    1750 4750
@@
 F 0 "R6" V 10050 3400 50  0000 C CNN
 F 1 "10k" V 9850 3400 50  0000 C CNN
-F 2 "" H 9950 3400 50  0001 C CNN
+F 2 "Resistor_SMD:R_0402_1005Metric" H 9950 3400 50  0001 C CNN
 F 3 "~" H 9950 3400 50  0001 C CNN
 	1    9950 3400
@@
 F 0 "SW6" H 10250 3600 50  0000 C CNN
 F 1 "SW_SPDT" H 10250 3200 50  0000 C CNN
-F 2 "" H 10250 3400 50  0001 C CNN
+F 2 "Button_Switch_SMD:SW_SPDT_PCM12" H 10250 3400 50  0001 C CNN
 F 3 "~" H 10250 3400 50  0001 C CNN
 	1    10250 3400
@@
 F 0 "SW5" H 10250 2850 50  0000 C CNN
 F 1 "SW_SPDT" H 10250 2450 50  0000 C CNN
-F 2 "" H 10250 2650 50  0001 C CNN
+F 2 "Button_Switch_SMD:SW_SPDT_PCM12" H 10250 2650 50  0001 C CNN
 F 3 "~" H 10250 2650 50  0001 C CNN
 	1    10250 2650
@@
 F 0 "R5" V 10050 2650 50  0000 C CNN
 F 1 "10k" V 9850 2650 50  0000 C CNN
-F 2 "" H 9950 2650 50  0001 C CNN
+F 2 "Resistor_SMD:R_0402_1005Metric" H 9950 2650 50  0001 C CNN
 F 3 "~" H 9950 2650 50  0001 C CNN
 	1    9950 2650
@@
 F 0 "R0" V 1300 3000 50  0000 C CNN
 F 1 "10k" V 1100 3000 50  0000 C CNN
-F 2 "" H 1200 3000 50  0001 C CNN
+F 2 "Resistor_SMD:R_0402_1005Metric" H 1200 3000 50  0001 C CNN
 F 3 "~" H 1200 3000 50  0001 C CNN
 	1    1200 3000
@@
 F 0 "SW0" H 1500 3200 50  0000 C CNN
 F 1 "SW_SPDT" H 1500 2800 50  0000 C CNN
-F 2 "" H 1500 3000 50  0001 C CNN
+F 2 "Button_Switch_SMD:SW_SPDT_PCM12" H 1500 3000 50  0001 C CNN
 F 3 "~" H 1500 3000 50  0001 C CNN
 	1    1500 3000
